File: Schematics KiCad FIles/Blowout_Control_Unit_441C801/Blowout_Control_Unit_441C801.kicad_sch (KiCad schematic)
At the start: 11 parts, among them U1 5963

Commit message: 2026/3/3
Parts:
- added C10, C6, C9: 25pF, symbol Device:C
- added C4, C8: 150pF, symbol Device:C
- added C5, C7: 100pF, symbol Device:C
- added R10, R12, R18, R23: 360k, symbol Device:R
- added R11, R19, R22, R9: 1k, symbol Device:R
- added R13, R17, R24, R8: 390k, symbol Device:R
- added R14, R15, R20, R21: 33k, symbol Device:R
- added R16, R25, R26: 47k, symbol Device:R
- added U2, U3: 5963, Valve:Valve_Noval_P, symbol Valve:ECC81
Connections:
- net +200V: now also R14.1, R15.1, R20.1, R21.1
- net GND: now also U2.3 (K), U2.8 (K), U3.3 (K), U3.8 (K)
- net at R7.2: now also C3.1
- net at C3.2: now also C4.1, R10.2, R8.2, R9.1
- new net: C8.1, R20.2, R24.2, U3.1 (A)
- new net: C8.2, R22.2, R23.2, R24.1, R25.1
- new net: C6.2, C7.1, R17.2, R18.2, R19.1
- new net: C7.2, R17.1, R21.2, U3.6 (A)
- new net: C5.2, C9.2, R11.2, R12.2, R13.1
- new net: C5.1, R13.2, R14.2, R16.1, U2.1 (A)
- new net: C9.1, R26.2
- new net: R9.2, U2.2 (G)
- new net: C4.2, R15.2, R8.1, U2.6 (A)
- new net: R19.2, U3.2 (G)
- new net: R11.1, U2.7 (G)
- new net: R22.1, U3.7 (G)
- new net: C6.1, R16.2
- new net: C10.1, R25.2
- new net -105V: R10.1, R12.1, R18.1, R23.1
- new net Clock Pulses (-): C10.2, R26.1
Other:
- note added: "1ST DELAY FLIP FLOP"
- note added: "2ND DELAY FLIP FLOP"
- note added: "SHIFT PULSE SHAPER"

Commit message: 2026/3/3
Parts:
- added C11: 250pF, symbol Device:C
- added C12, C13, C14: 25pF, symbol Device:C
- added J1: Conn_02x12_Top_Bottom, symbol Connector_Generic:Conn_02x12_Top_Bottom
- added R27: 10k, symbol Device:R
- added R28, R30, R31, R33: 47k, symbol Device:R
- added R29: 470k, symbol Device:R
- added R32, R34, R35: 220k, symbol Device:R
- added U4, U5: 5963, Valve:Valve_Noval_P, symbol Valve:ECC81
Connections:
- net +200V: now also J1.17 (Pin_17), R28.1, U4.1 (A)
- net +75V: now also J1.2 (Pin_2)
- net -105V: now also J1.6 (Pin_6)
- net -30V: now also J1.14 (Pin_14), R32.1, R34.1, R35.1
- net Clock Pulses (-): now also J1.8 (Pin_8)
- net GND: now also J1.1 (Pin_1), R27.2, R29.1, U4.8 (K), U5.3 (K), U5.8 (K)
- net Shift Pulse Input: now also J1.3 (Pin_3)
- net Shift Pulse Out to M'plier: now also J1.15 (Pin_15)
- net at C7.2, R17.1, R21.2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: now also R30.1, R31.1
- net at C5.1, R13.2, R14.2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: now also R33.1
- net FIL. PIN 4,5: now reaches U3.4 (F1)
- net FIL. PIN 4,5: now also U1.4 (F1), U1.5 (F1), U2.4 (F1), U2.5 (F1), U3.5 (F1), J1.12 (Pin_12), U4.4 (F1), U4.5 (F1), U5.4 (F1), U5.5 (F1)
- net FIL. PIN 9: now reaches U3.9 (F2)
- net FIL. PIN 9: now also U1.9 (F2), U2.9 (F2), J1.24 (Pin_24), U4.9 (F2), U5.9 (F2)
- new net: C14.1, R35.2, U5.7 (G)
- new net: C13.2, R31.2
- new net: C12.1, R32.2, U4.7 (G)
- new net: C11.1, R29.2, U4.2 (G)
- new net: C13.1, R34.2, U5.2 (G)
- new net: C12.2, R33.2
- new net: C11.2, R30.2
- new net M'CAND RING BLOWOUT: J1.21 (Pin_21), R28.2, U4.6 (A), U5.1 (A), U5.6 (A)
- new net M'CAND TALLY IN: C14.2, J1.22 (Pin_22)
- new net XO OUT: J1.10 (Pin_10), R27.1, U4.3 (K)
Other:
- note added: "XO CF BUFF."
- moved on the sheet: U1C, U2C, U3C
