File: Schematics KiCad FIles/Accumulator_Unit_441C1201/flip_flop_4.kicad_sch (KiCad schematic)
At the start: 16 parts, among them U1204 5963, U1205 6BC7

Commit message: Fix component designators on accumulator schematics
Parts:
- renumbered R17 to AB17, R47 to AB47, R48 to AB48, R18 to CD18, C19 to CD19, R20 to CD20, C21 to CD21, R22 to CD22, R23 to CD23, C24 to CD24, R43 to CD43, C44 to CD44, R45 to CD45, C46 to CD46, U1204 to V1204, U1205 to V1205
Changed lines of the file:
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@@
 		(on_board yes)
 		(dnp no)
-		(property "Reference" "C21"
+		(property "Reference" "CD21"
 			(at 149.86 77.4699 0)
 			(effects
@@
 			(project "Accumulator_Unit_441C1201"
 				(path "/519d7692-6bf3-45ab-bd58-713783b63e8a/bbd7ed54-3527-4ba8-b036-f61fa03898f2"
-					(reference "C21")
+					(reference "CD21")
 					(unit 1)
 				)
@@
 		(on_board yes)
 		(dnp no)
-		(property "Reference" "R17"
+		(property "Reference" "AB17"
 			(at 72.39 59.6899 0)
 			(effects
@@
 			(project "Accumulator_Unit_441C1201"
 				(path "/519d7692-6bf3-45ab-bd58-713783b63e8a/bbd7ed54-3527-4ba8-b036-f61fa03898f2"
-					(reference "R17")
+					(reference "AB17")
 					(unit 1)
 				)
@@
 		(on_board yes)
 		(dnp no)
-		(property "Reference" "R45"
+		(property "Reference" "CD45"
 			(at 72.39 97.7899 0)
 			(effects
@@
 			(project "Accumulator_Unit_441C1201"
 				(path "/519d7692-6bf3-45ab-bd58-713783b63e8a/bbd7ed54-3527-4ba8-b036-f61fa03898f2"
-					(reference "R45")
+					(reference "CD45")
 					(unit 1)
 				)
@@
 		(on_board yes)
 		(dnp no)
-		(property "Reference" "R18"
+		(property "Reference" "CD18"
 			(at 135.89 97.7899 0)
 			(effects
@@
 			(project "Accumulator_Unit_441C1201"
 				(path "/519d7692-6bf3-45ab-bd58-713783b63e8a/bbd7ed54-3527-4ba8-b036-f61fa03898f2"
-					(reference "R18")
+					(reference "CD18")
 					(unit 1)
 				)
@@
 		(on_board yes)
 		(dnp no)
-		(property "Reference" "R43"
+		(property "Reference" "CD43"
 			(at 72.39 77.4699 0)
 			(effects
@@
 			(project "Accumulator_Unit_441C1201"
 				(path "/519d7692-6bf3-45ab-bd58-713783b63e8a/bbd7ed54-3527-4ba8-b036-f61fa03898f2"
-					(reference "R43")
+					(reference "CD43")
 					(unit 1)
 				)
@@
 		(on_board yes)
 		(dnp no)
-		(property "Reference" "R48"
+		(property "Reference" "AB48"
 			(at 161.29 77.4699 0)
 			(effects
@@
 			(project "Accumulator_Unit_441C1201"
 				(path "/519d7692-6bf3-45ab-bd58-713783b63e8a/bbd7ed54-3527-4ba8-b036-f61fa03898f2"
-					(reference "R48")
+					(reference "AB48")
 					(unit 1)
 				)
@@
 		(on_board yes)
 		(dnp no)
-		(property "Reference" "C24"
+		(property "Reference" "CD24"
 			(at 255.27 101.5999 0)
 			(effects
@@
 			(project "Accumulator_Unit_441C1201"
 				(path "/519d7692-6bf3-45ab-bd58-713783b63e8a/bbd7ed54-3527-4ba8-b036-f61fa03898f2"
-					(reference "C24")
+					(reference "CD24")
 					(unit 1)
 				)
@@
 		(dnp no)
 		(fields_autoplaced yes)
-		(property "Reference" "U1205"
+		(property "Reference" "V1205"
 			(at 238.76 76.194 0)
 			(effects
@@
 			(project ""
 				(path "/519d7692-6bf3-45ab-bd58-713783b63e8a/bbd7ed54-3527-4ba8-b036-f61fa03898f2"
-					(reference "U1205")
+					(reference "V1205")
 					(unit 1)
 				)
@@
 		(on_board yes)
 		(dnp no)
-		(property "Reference" "U1204"
+		(property "Reference" "V1204"
 			(at 113.03 87.6299 0)
 			(effects
@@
 			(project "Accumulator_Unit_441C1201"
 				(path "/519d7692-6bf3-45ab-bd58-713783b63e8a/bbd7ed54-3527-4ba8-b036-f61fa03898f2"
-					(reference "U1204")
+					(reference "V1204")
 					(unit 1)
 				)
@@
 		(on_board yes)
 		(dnp no)
-		(property "Reference" "C44"
+		(property "Reference" "CD44"
 			(at 58.42 77.4699 0)
 			(effects
@@
 			(project "Accumulator_Unit_441C1201"
 				(path "/519d7692-6bf3-45ab-bd58-713783b63e8a/bbd7ed54-3527-4ba8-b036-f61fa03898f2"
-					(reference "C44")
+					(reference "CD44")
 					(unit 1)
 				)
@@
 		(dnp no)
 		(fields_autoplaced yes)
-		(property "Reference" "U1204"
+		(property "Reference" "V1204"
 			(at 95.25 87.6299 0)
 			(effects
@@
 			(project "Accumulator_Unit_441C1201"
 				(path "/519d7692-6bf3-45ab-bd58-713783b63e8a/bbd7ed54-3527-4ba8-b036-f61fa03898f2"
-					(reference "U1204")
+					(reference "V1204")
 					(unit 2)
 				)
@@
 		(on_board yes)
 		(dnp no)
-		(property "Reference" "C46"
+		(property "Reference" "CD46"
 			(at 58.42 97.7899 0)
 			(effects
@@
 			(project "Accumulator_Unit_441C1201"
 				(path "/519d7692-6bf3-45ab-bd58-713783b63e8a/bbd7ed54-3527-4ba8-b036-f61fa03898f2"
-					(reference "C46")
+					(reference "CD46")
 					(unit 1)
 				)
@@
 		(on_board yes)
 		(dnp no)
-		(property "Reference" "R23"
+		(property "Reference" "CD23"
 			(at 254 54.6099 0)
 			(effects
@@
 			(project "Accumulator_Unit_441C1201"
 				(path "/519d7692-6bf3-45ab-bd58-713783b63e8a/bbd7ed54-3527-4ba8-b036-f61fa03898f2"
-					(reference "R23")
+					(reference "CD23")
 					(unit 1)
 				)
@@
 		(dnp no)
 		(fields_autoplaced yes)
-		(property "Reference" "U1204"
+		(property "Reference" "V1204"
 			(at 127 160.0199 0)
 			(effects
@@
 			(project "Accumulator_Unit_441C1201"
 				(path "/519d7692-6bf3-45ab-bd58-713783b63e8a/bbd7ed54-3527-4ba8-b036-f61fa03898f2"
-					(reference "U1204")
+					(reference "V1204")
 					(unit 3)
 				)
@@
 		(dnp no)
 		(fields_autoplaced yes)
-		(property "Reference" "U1205"
+		(property "Reference" "V1205"
 			(at 151.13 160.0199 0)
 			(effects
@@
 			(project ""
 				(path "/519d7692-6bf3-45ab-bd58-713783b63e8a/bbd7ed54-3527-4ba8-b036-f61fa03898f2"
-					(reference "U1205")
+					(reference "V1205")
 					(unit 2)
 				)
@@
 		(on_board yes)
 		(dnp no)
-		(property "Reference" "R22"
+		(property "Reference" "CD22"
 			(at 219.71 54.6099 0)
 			(effects
@@
 			(project "Accumulator_Unit_441C1201"
 				(path "/519d7692-6bf3-45ab-bd58-713783b63e8a/bbd7ed54-3527-4ba8-b036-f61fa03898f2"
-					(reference "R22")
+					(reference "CD22")
 					(unit 1)
 				)
@@
 		(on_board yes)
 		(dnp no)
-		(property "Reference" "C19"
+		(property "Reference" "CD19"
 			(at 149.86 97.7899 0)
 			(effects
@@
 			(project "Accumulator_Unit_441C1201"
 				(path "/519d7692-6bf3-45ab-bd58-713783b63e8a/bbd7ed54-3527-4ba8-b036-f61fa03898f2"
-					(reference "C19")
+					(reference "CD19")
 					(unit 1)
 				)
@@
 		(on_board yes)
 		(dnp no)
-		(property "Reference" "R20"
+		(property "Reference" "CD20"
 			(at 135.89 77.4699 0)
 			(effects
@@
 			(project "Accumulator_Unit_441C1201"
 				(path "/519d7692-6bf3-45ab-bd58-713783b63e8a/bbd7ed54-3527-4ba8-b036-f61fa03898f2"
-					(reference "R20")
+					(reference "CD20")
 					(unit 1)
 				)
@@
 		(on_board yes)
 		(dnp no)
-		(property "Reference" "R47"
+		(property "Reference" "AB47"
 			(at 135.89 59.6899 0)
 			(effects
@@
 			(project "Accumulator_Unit_441C1201"
 				(path "/519d7692-6bf3-45ab-bd58-713783b63e8a/bbd7ed54-3527-4ba8-b036-f61fa03898f2"
-					(reference "R47")
-					(unit 1)
-				)
+					(reference "AB47")
+					(unit 1)
+				)
